File: KiCad v0.3 (controller + battery)/TestWatch.kicad_sch (KiCad schematic)
At the start: 206 parts, among them IC1 STM32G431KBT6, J1 Conn_01x08, J2 Conn_01x08, J3 Conn_01x08, J4 Conn_01x08

Commit message: Uhm
Parts:
- removed D1, D10, D100, D101, D102, D103, D104, D105, D106, D107, D108, D109, D11, D110, D111, D112, D113, D114, D115, D116, D117, D118, D119, D12, D120, D121, D122, D123, D124, D125, D126, D127, D128, D129, D13, D130, D131, D132, D133, D134, D135, D136, D137, D138, D139, D14, D140, D141, D142, D143, D144, D145, D146, D147, D148, D149, D15, D150, D151, D152, D153, D154, D155, D156, D157, D158, D159, D16, D160, D161, D162, D163, D164, D165, D166, D167, D168, D169, D17, D170, D171, D172, D173, D174, D175, D176, D177, D178, D179, D18, D180, D181, D182, D183, D184, D185, D186, D187, D188, D189, D19, D190, D191, D192, D193, D194, D195, D196, D197, D198, D199, D2, D20, D200, D201, D21, D22, D23, D24, D25, D26, D27, D28, D29, D3, D30, D31, D32, D33, D34, D35, D36, D37, D38, D39, D4, D40, D41, D42, D43, D44, D45, D46, D47, D48, D49, D5, D50, D51, D52, D53, D54, D55, D56, D57, D58, D59, D6, D60, D61, D62, D63, D64, D65, D66, D67, D68, D69, D7, D70, D71, D72, D73, D74, D75, D76, D77, D78, D79, D8, D80, D81, D82, D83, D84, D85, D86, D87, D88, D89, D9, D90, D91, D92, D93, D94, D95, D96, D97, D98, D99: WL-SMCC_0402, WL-SMCC_0402:WL-SMCC_0402, symbol WL-SMCC_0402:WL-SMCC_0402
- removed J1, J2, J3, J4: Conn_01x08, symbol Connector_Generic:Conn_01x08
- added BT1: BAT-HLD-003-SMT, BAT-HLD-003-SMT:BAT_BAT-HLD-003-SMT_CUT, symbol BAT-HLD-003-SMT_CUT:BAT-HLD-003-SMT
- added BUTT1: B3U-1100P, B3U_1100P:SW_B3U-1100P, symbol B3U-1100P:B3U-1100P
- added C1: GRM21BC81E106ME51K, GRM21BC81E106ME51K:CAPC2012X140N, symbol GRM21BC81E106ME51K:GRM21BC81E106ME51K
- added CHG1: MCP73832T-2ACI_OT, MCP73832T_2ACI_OT:SOT95P270X145-5N, symbol MCP73832T-2ACI_OT:MCP73832T-2ACI_OT
- added CUT1: MAX809SEUR_T, MAX809SEUR+T:MAX809SEUR+T, symbol MAX809SEUR_T:MAX809SEUR_T
- added J1: Conn_01x16, Connector_PinSocket_2.54mm:PinSocket_1x16_P2.54mm_Vertical, symbol Connector_Generic:Conn_01x16
- added Osc1: MC-306_32.7680K-E0_PURE_SN, MC-306_32.7680K-E0_PURE_SN:MC-306_32.7680K-E0_PURE_SN, symbol MC-306_32.7680K-E0_PURE_SN:MC-306_32.7680K-E0_PURE_SN
- added P13, P14: ~, WL-SMCC_0402:PROGPAD, symbol PGO:PROGPAD
- added POGO1: ~, WL-SMCC_0402:Untitled, symbol PGO:POGO_FEMALE_2
- added Q1: IRLML6402, Package_TO_SOT_SMD:SOT-23, symbol Transistor_FET:IRLML6402
- added R1, R2, R3: RN73H1JTTD5052F50, RN73H1JTTD5052F50:RN73H1JTTD5052F50, symbol RN73H1JTTD5052F50:RN73H1JTTD5052F50
- added REG1: TPS7A0225PDBVR, TPS7A0225PDBVR:TPS7A0225PDBVR, symbol TPS7A0225PDBVR:TPS7A0225PDBVR
- STM1: renamed from IC1; footprint QFP80P900X900X160-32N -> STM32G431KBT6:QFP80P900X900X160-32N
Connections:
- net A: now also STM1.7 (PA2), J1.1 (Pin_1)
- net B: now also STM1.8 (PA3), J1.2 (Pin_2)
- net C: now also STM1.9 (PA4), J1.3 (Pin_3)
- net D: now also STM1.10 (PA5), J1.4 (Pin_4)
- net E: now also STM1.11 (PA6), J1.5 (Pin_5)
- net F: now also STM1.12 (PA7), J1.6 (Pin_6)
- net G: now also STM1.18 (PA8), J1.7 (Pin_7)
- net H: now also STM1.19 (PA9), J1.8 (Pin_8)
- net I: now also STM1.20 (PA10), J1.9 (Pin_9)
- net J: now also STM1.21 (PA11), J1.10 (Pin_10)
- net K: now also STM1.22 (PA12), J1.11 (Pin_11)
- net L: now also STM1.25 (PA15), J1.12 (Pin_12)
- net M: now also STM1.26 (PB3), J1.13 (Pin_13)
- net N: now also STM1.27 (PB4), J1.14 (Pin_14)
- net O: now also STM1.28 (PB5), J1.15 (Pin_15)
- net P: now also STM1.29 (PB6), J1.16 (Pin_16)
- net at STM1.13 (PB0): now also Q1.1 (G), R3.2
- net GNDREF: now reaches STM1.14 (VSSA)
- net GNDREF: now also STM1.16 (VSS_1), STM1.31 (PB8-BOOT0), STM1.32 (VSS_2), BT1.N, C1.2, CHG1.2 (VSS), CUT1.1 (GND), POGO1.2 (USB_-), R1.2, R2.2, REG1.2 (GND)
- net STM_POW: now reaches STM1.15 (VDDA)
- net STM_POW: now also STM1.1 (VDD_1), STM1.17 (VDD_2), STM1.6 (PA1), BUTT1.2, REG1.5 (OUT)
- net at STM1.2 (PF0-OSC_IN): now also Osc1.1
- net at STM1.3 (PF1-OSC_OUT): now also Osc1.4
- net at STM1.5 (PA0): now also BUTT1.1, R2.1
- net at STM1.23 (PA13): now also P14.1
- net at STM1.24 (PA14): now also P13.1
- new net: C1.1, CHG1.4 (VDD), Q1.3 (D)
- new net: CHG1.5 (PROG), R1.1
- new net: CUT1.2 (~{RESET}), REG1.3 (EN)
- new net: Osc1.2 (NC), Osc1.3 (NC__1)
- new net BATT: BT1.P1, BT1.P2, CHG1.3 (VBAT), CUT1.3 (VCC), REG1.1 (IN)
- new net USB + : POGO1.1 (USB_+), Q1.2 (S), R3.1
Other:
- note added: "Drain"
- note added: "Gate"
- note added: "Source"
- moved on the sheet: STM1

Commit message: v0.3 sent for fab, v0.4 still in progress
v0.3 and v0.4 have the same component footprints - that way, I only need to have 1 stencil (if v0.3 works!!!)
Parts:
- removed CUT1: MAX809SEUR_T, MAX809SEUR+T:MAX809SEUR+T, symbol MAX809SEUR_T:MAX809SEUR_T
- removed Osc1: MC-306_32.7680K-E0_PURE_SN, MC-306_32.7680K-E0_PURE_SN:MC-306_32.7680K-E0_PURE_SN, symbol MC-306_32.7680K-E0_PURE_SN:MC-306_32.7680K-E0_PURE_SN
- removed Q1: IRLML6402, Package_TO_SOT_SMD:SOT-23, symbol Transistor_FET:IRLML6402
- removed R3: RN73H1JTTD5052F50, RN73H1JTTD5052F50:RN73H1JTTD5052F50, symbol RN73H1JTTD5052F50:RN73H1JTTD5052F50
- removed REG1: TPS7A0225PDBVR, TPS7A0225PDBVR:TPS7A0225PDBVR, symbol TPS7A0225PDBVR:TPS7A0225PDBVR
- added C2, C3: GRM21BC81E106ME51K, GRM21BC81E106ME51K:CAPC2012X140N, symbol GRM21BC81E106ME51K:GRM21BC81E106ME51K
- added DB1, DB2: BAS3010A03WE6327HTSA1, BAS3010A03WE6327HTSA1:SOD2513X110N, symbol BAS3010A03WE6327HTSA1:BAS3010A03WE6327HTSA1
- added DB3: 1N4148WT, Diode_SMD:D_SOD-523, symbol Diode:1N4148WT
- added J2: Conn_01x04, Connector_PinHeader_2.54mm:PinHeader_1x04_P2.54mm_Vertical, symbol Connector_Generic:Conn_01x04
- added OSC1: MC-306_32.7680K-E0_PURE_SN, MC-306_32.7680K-E0_PURE_SN:MC-306_32.7680K-E0_PURE_SN, symbol MC-306_32.7680K-E0_PURE_SN:MC-306_32.7680K-E0_PURE_SN
- added R3: RC1206FR-07120KL, RC1206FR_07120KL:RC1206FR_07120KL, symbol RC1206FR-07120KL:RC1206FR-07120KL
- added R4: RMCF0603FT300K, RMCF0603FT300K:RMCF0603FT300K, symbol RMCF0603FT300K:RMCF0603FT300K
- added R5: RN73H1JTTD5052F50, RN73H1JTTD5052F50:RN73H1JTTD5052F50, symbol RN73H1JTTD5052F50:RN73H1JTTD5052F50
- added R6: RC1005F103CS, RC1005F103CS:RESC1005X40N, symbol RC1005F103CS:RC1005F103CS
- added U1: TPS7A0230PDBVR, TPS7A0230PDBVR:TPS7A0230PDBVR, symbol TPS7A0230PDBVR:TPS7A0230PDBVR
- J1: footprint Connector_PinSocket_2.54mm:PinSocket_1x16_P2.54mm_Vertical -> Connector_PinHeader_2.54mm:PinHeader_1x16_P2.54mm_Vertical
- renumbered P14 to P13, P13 to P14
Connections:
- net G: now also STM1.13 (PB0); no longer STM1.18 (PA8)
- net GNDREF: now also C2.2, C3.2, J2.4 (Pin_4), R4.2, U1.2 (GND)
- net H: now also STM1.18 (PA8); no longer STM1.19 (PA9)
- net I: now also STM1.19 (PA9); no longer STM1.20 (PA10)
- net J: now also STM1.20 (PA10); no longer STM1.21 (PA11)
- net K: now also STM1.21 (PA11); no longer STM1.22 (PA12)
- net L: now also STM1.22 (PA12); no longer STM1.25 (PA15)
- net M: now also STM1.25 (PA15); no longer STM1.26 (PB3)
- net N: now also STM1.28 (PB5); no longer STM1.27 (PB4)
- net O: now also STM1.29 (PB6); no longer STM1.28 (PB5)
- net P: now also STM1.30 (PB7); no longer STM1.29 (PB6)
- net STM_POW: now also C2.1, J2.1 (Pin_1), R6.2, U1.5 (OUT); no longer STM1.6 (PA1)
- net USB + : now also C1.1, CHG1.4 (VDD), DB1.A, R5.2
- net at CHG1.1 (STAT): now also DB3.1 (K), R5.1
- net at P13.1, STM1.23 (PA13): now also J2.3 (Pin_3)
- net at STM1.2 (PF0-OSC_IN): now also OSC1.4
- net at P14.1, STM1.24 (PA14): now also J2.2 (Pin_2)
- net at STM1.3 (PF1-OSC_OUT): now also OSC1.1
- net at STM1.4 (PG10-NRST): now also R6.1
- removed net BATT: BT1.P1, BT1.P2, CHG1.3 (VBAT)
- new net: BT1.P, C3.1, CHG1.3 (VBAT), R3.1, U1.1 (IN)
- new net: DB3.2 (A), STM1.27 (PB4)
- new net: DB1.C, DB2.C, U1.3 (EN)
- new net: DB2.A, STM1.26 (PB3)
- new net: R3.2, R4.1, STM1.6 (PA1)
- no-connect marks 0 -> 1
Other:
- note added: "3.3V"
- note added: "5V+"
- note added: "A"
- note added: "C"
- note added: "STM32"
- note removed: "Drain"
- note removed: "Gate"
- note removed: "Source"
- moved on the sheet: BUTT1, C1, CHG1, P13, P14, POGO1, R1, R2
