File: Hardware/Complete v3.0/Complete v3.0.kicad_pcb (KiCad board)
At the start: 4 copper layers, 37 x 37 mm, 221 parts, among them Q1 SI2301DS, U1 TPS7A0230PDBVR, U2 ATMEGA4808-AU, U3 DS3231MZ_

Commit message: Version 3 software update
• set the BOD to 2.6V (dont go higher than that)

• Added charger wake flag

• Added charger indicator

• Set the software version number to match the hardware number
Other:
- board text added: "Follow schematic guidance"
- board text removed: "Line on component goes here"
Changed lines of the file:
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@@
 		)
 	)
-	(gr_text "Line on component goes here"
+	(gr_text "Follow schematic guidance"
 		(at 238.5 106.5 0)
 		(layer "User.1")

Commit message: Near Final Update
Found out the BOD controller only shuts down the chip control instead of shutting down the functionality of the pins. I have rewrote the software to use a different control function (VLM instead of BOD) so it should (in theory) be able to shut down safely.

Additionally, I re-wired 2 traces on the circuit board so that the battery-percentage module is 100% safe and will not drain the battery. It's not worth paying the money to get new boards printed, since there's only one non-critical wire added to the back of the board. If the wire breaks contact, the battery read module will read 99% since there's no "ground" connected.

This needs to be tested, of course.
Other:
- board text added: "Removed resistor for testing bat life after 0 charge"
Changed lines of the file:
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@@
 	)
 	(gr_line
+		(start 206 102)
+		(end 212.5 90.5)
+		(stroke
+			(width 0.1)
+			(type default)
+		)
+		(layer "User.1")
+	)
+	(gr_line
 		(start 244 85.5)
 		(end 226 85.5)
@@
 		)
 	)
+	(gr_text "Removed resistor for \ntesting bat life after \n0 charge\n"
+		(at 199 108 0)
+		(layer "User.1")
+		(effects
+			(font
+				(size 1 1)
+				(thickness 0.15)
+			)
+			(justify left bottom)
+		)
+	)
